Commit message: camara gazebo lista

File: robots/kobuki_hexagons_rplidar.urdf.xacro (robot description, xacro)
@@ -18,5 +18,5 @@
   </xacro:rplidar>
   <xacro:generic_camera parent="base_link" name="camera">
-  		<origin xyz="0.1 0 0.420" rpy="3.1415 0 1.5707"/>
+  		<origin xyz="0.13 0 0.400" rpy="0 0.78535 0"/>
   </xacro:generic_camera>
 </robot>

File: urdf/sensors/camera.urdf.xacro (robot description, xacro)
@@ -18,8 +18,8 @@
         <origin xyz="0 0 0" rpy="0 0 0" />
         <geometry>
-          <box size="0.01 0.01 0.01" />
+          <box size="0.02 0.02 0.02" />
         </geometry>
-        <material name="grey">
-            <color rgba="0.2 0.2 0.2 1.0"/>
+        <material name="Cyan">
+          <color rgba="0 1.0 1.0 1.0"/>
         </material>
       </visual>
@@ -39,10 +39,10 @@
         <update_rate>30.0</update_rate>
         <camera>
-          <pose>0.035 0 0.078 0 ${-M_PI/2} 0</pose>
+          <!--<pose>0.035 0 0.078 0 ${-M_PI/2} 0</pose>-->
           <horizontal_fov>${85 * M_PI/180.0}</horizontal_fov>
           <image>
             <format>R8G8B8</format>
-            <width>1020</width>
-            <height>1020</height>
+            <width>800</width>
+            <height>600</height>
           </image>
           <clip>
